File: pbm_driver4.kicad_sch (KiCad schematic)
At the start: 0 parts

Commit message: As released to fab PCB103_RevA
Parts:
- added H1, H2, H3, H4: MountingHole_Pad, $Local:MountingHole_3.2mm_M3_Pad, symbol Mechanical:MountingHole_Pad
- added J1: Conn_02x10_Odd_Even, $Local:PinHeader_2x10_P2.54mm_Vertical, symbol Connector_Generic:Conn_02x10_Odd_Even
- added J2: Conn_01x10, $Local:PinHeader_1x10_P2.54mm_Vertical, symbol Connector_Generic:Conn_01x10
Connections:
- new net +12V: J1.2 (Pin_2), J2.2 (Pin_2), J2.4 (Pin_4), J2.6 (Pin_6), J2.8 (Pin_8)
- new net +3.3V: J1.20 (Pin_20)
- new net DAC1: J1.3 (Pin_3)
- new net DAC2: J1.4 (Pin_4)
- new net GND: H1.1, H2.1, H3.1, H4.1, J1.1 (Pin_1), J1.10 (Pin_10), J1.15 (Pin_15), J1.16 (Pin_16), J1.19 (Pin_19), J1.9 (Pin_9), J2.1 (Pin_1), J2.10 (Pin_10)
- new net I2C_SCL: J1.17 (Pin_17)
- new net I2C_SDA: J1.18 (Pin_18)
- new net LED1: J2.3 (Pin_3)
- new net LED2: J2.5 (Pin_5)
- new net LED3: J2.7 (Pin_7)
- new net LED4: J2.9 (Pin_9)
- new net SEL1: J1.11 (Pin_11)
- new net SEL2: J1.12 (Pin_12)
- new net SEL3: J1.13 (Pin_13)
- new net SEL4: J1.14 (Pin_14)
- new net SENSE1: J1.5 (Pin_5)
- new net SENSE2: J1.6 (Pin_6)
- new net SENSE3: J1.7 (Pin_7)
- new net SENSE4: J1.8 (Pin_8)
Other:
- removed sheet Sheet 3
- removed sheet Sheet 4
- sheet Sheet 5 ports: added I2C_SCL, I2C_SDA; removed none
