File: sheet2.kicad_sch (KiCad schematic)
At the start: 22 parts, among them Q1 PSMN4R0-30YLD, Q2 PSMN4R0-30YLD, Q3 PSMN4R0-30YLD, Q4 PSMN4R0-30YLD, U1 ADA4099-2, U2 ADA4099-2, U21 TMUX1112PWR

Commit message: As released to fab PCB103_RevA
Parts:
- C1, C2: value 1nF -> 0.1uF; footprint Capacitor_SMD:C_0603_1608Metric -> $Local:C_0603_1608Metric
- C21: value 1nF -> 0.1uF; footprint Capacitor_SMD:C_0603_1608Metric_Pad1.08x0.95mm_HandSolder -> $Local:C_0603_1608Metric
- Q1, Q2, Q3, Q4: footprint Package_TO_SOT_SMD:LFPAK56 -> $Local:LFPAK56
- R1, R2, R3, R4: footprint Resistor_SMD:R_1210_3225Metric_Pad1.30x2.65mm_HandSolder -> $Local:R_1210_3225Metric_Pad1.30x2.65mm_HandSolder
- R11, R12, R13, R14, R21, R22, R23, R24: footprint Resistor_SMD:R_0603_1608Metric_Pad0.98x0.95mm_HandSolder -> $Local:R_0603_1608Metric
- U1, U2: footprint Package_SO:SOIC-8_3.9x4.9mm_P1.27mm -> $Local:SOIC-8_3.9x4.9mm_P1.27mm
