File: sheet5.kicad_sch (KiCad schematic)
At the start: 5 parts, among them Q9 MMBT3906, U12 D36V6F5, U5 STM32G431RBTx, U6 LP2985-3.3, U8 TMP422

Commit message: As released to fab PCB103_RevA
Parts:
- removed Q9: MMBT3906, Package_TO_SOT_SMD:SOT-23, symbol Transistor_BJT:MMBT3906
- removed U12: D36V6F5, $Local:D36V6F5, symbol $Local:D36V6F5
- removed U5: STM32G431RBTx, Package_QFP:LQFP-64_10x10mm_P0.5mm, symbol MCU_ST_STM32G4:STM32G431RBTx
- removed U6: LP2985-3.3, Package_TO_SOT_SMD:SOT-23-5, symbol Regulator_Linear:LP2985-3.3
- removed U8: TMP422, Package_TO_SOT_SMD:SOT-23-8, symbol $Local:TMP422
- added C13: 100pF, $Local:C_0805_2012Metric, symbol Device:C
- added C21 (x8): 10uF, $Local:C_0805_2012Metric, symbol Device:C
- added C21: 0.1uF, $Local:C_0603_1608Metric, symbol Device:C
- added Q5: MMBT3906, $Local:SOT-323_SC-70, symbol Transistor_BJT:MMBT3906
- added R10, R5, R6, R7, R8, R9: 10K, $Local:R_0603_1608Metric, symbol Device:R_US
- added U3: TMP421, $Local:SOT-23-8, symbol $Local:TMP421
Connections:
- new net +12V: C21.1, C21.1, C21.1, C21.1, C21.1, C21.1, C21.1, C21.1
- new net +3.3V: C21.1, R10.1, R5.1, R7.1, R9.1, U3.8 (V+)
- new net A0: R7.2, R8.1, U3.4 (A0)
- new net A1: R5.2, R6.1, U3.3 (A1)
- new net DX_N: C13.2, Q5.1 (B), U3.2 (DXN)
- new net DX_P: C13.1, Q5.2 (E), U3.1 (DXP)
- new net GND: C21.2, C21.2, C21.2, C21.2, C21.2, C21.2, C21.2, C21.2, C21.2, Q5.3 (C), R6.2, R8.2, U3.5 (GND)
- new net I2C_SCL: R9.2, U3.7 (SCL)
- new net I2C_SDA: R10.2, U3.6 (SDA)
Other:
- note added: "Check Footprint: 0805 or 0603?"
